File: reg_5v.kicad_sch (KiCad schematic)
At the start: 8 parts

Commit message: Finish schematic and start routing PCB
Parts:
- C11, C12, C13, C14: renamed from C?; footprint (none) -> Capacitor_SMD:C_0805_2012Metric_Pad1.18x1.45mm_HandSolder
- L2: renamed from L?; footprint (none) -> Inductor_SMD:L_0805_2012Metric_Pad1.15x1.40mm_HandSolder
- R11, R12: renamed from R?; footprint (none) -> Resistor_SMD:R_0805_2012Metric_Pad1.20x1.40mm_HandSolder
- U5: renamed from U?; footprint (none) -> Package_TO_SOT_SMD:SOT-23-6
Changed lines of the file:
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@@
   (symbol (lib_id "power:GND") (at 48.26 54.61 0) (unit 1)
     (in_bom yes) (on_board yes) (fields_autoplaced)
-    (property "Reference" "#PWR?" (id 0) (at 48.26 60.96 0)
+    (property "Reference" "#PWR034" (id 0) (at 48.26 60.96 0)
       (effects (font (size 1.27 1.27)) hide)
     )
@@
   (symbol (lib_id "power:GND") (at 66.04 54.61 0) (unit 1)
     (in_bom yes) (on_board yes) (fields_autoplaced)
-    (property "Reference" "#PWR?" (id 0) (at 66.04 60.96 0)
+    (property "Reference" "#PWR035" (id 0) (at 66.04 60.96 0)
       (effects (font (size 1.27 1.27)) hide)
     )
@@
   (symbol (lib_id "Device:C_Small") (at 50.8 43.18 0) (unit 1)
     (in_bom yes) (on_board yes) (fields_autoplaced)
-    (property "Reference" "C?" (id 0) (at 53.1241 42.3516 0)
+    (property "Reference" "C12" (id 0) (at 53.1241 42.3516 0)
       (effects (font (size 1.27 1.27)) (justify left))
     )
@@
       (effects (font (size 1.27 1.27)) (justify left))
     )
-    (property "Footprint" "" (id 2) (at 50.8 43.18 0)
+    (property "Footprint" "Capacitor_SMD:C_0805_2012Metric_Pad1.18x1.45mm_HandSolder" (id 2) (at 50.8 43.18 0)
       (effects (font (size 1.27 1.27)) hide)
     )
@@
   (symbol (lib_id "Device:L_Small") (at 110.49 31.75 90) (unit 1)
     (in_bom yes) (on_board yes)
-    (property "Reference" "L?" (id 0) (at 110.49 26.67 90))
+    (property "Reference" "L2" (id 0) (at 110.49 26.67 90))
     (property "Value" "4.7uH" (id 1) (at 110.49 29.21 90))
-    (property "Footprint" "" (id 2) (at 110.49 31.75 0)
+    (property "Footprint" "Inductor_SMD:L_0805_2012Metric_Pad1.15x1.40mm_HandSolder" (id 2) (at 110.49 31.75 0)
       (effects (font (size 1.27 1.27)) hide)
     )
@@
   (symbol (lib_id "Device:R_Small_US") (at 118.11 36.83 0) (unit 1)
     (in_bom yes) (on_board yes) (fields_autoplaced)
-    (property "Reference" "R?" (id 0) (at 119.761 35.9953 0)
+    (property "Reference" "R11" (id 0) (at 119.761 35.9953 0)
       (effects (font (size 1.27 1.27)) (justify left))
     )
@@
       (effects (font (size 1.27 1.27)) (justify left))
     )
-    (property "Footprint" "" (id 2) (at 118.11 36.83 0)
+    (property "Footprint" "Resistor_SMD:R_0805_2012Metric_Pad1.20x1.40mm_HandSolder" (id 2) (at 118.11 36.83 0)
       (effects (font (size 1.27 1.27)) hide)
     )
@@
   (symbol (lib_id "power:GND") (at 118.11 54.61 0) (unit 1)
     (in_bom yes) (on_board yes) (fields_autoplaced)
-    (property "Reference" "#PWR?" (id 0) (at 118.11 60.96 0)
+    (property "Reference" "#PWR036" (id 0) (at 118.11 60.96 0)
       (effects (font (size 1.27 1.27)) hide)
     )
@@
   (symbol (lib_id "Device:C_Small") (at 45.72 43.18 0) (unit 1)
     (in_bom yes) (on_board yes)
-    (property "Reference" "C?" (id 0) (at 39.37 43.18 0)
+    (property "Reference" "C11" (id 0) (at 39.37 43.18 0)
       (effects (font (size 1.27 1.27)) (justify left))
     )
@@
       (effects (font (size 1.27 1.27)) (justify left))
     )
-    (property "Footprint" "" (id 2) (at 45.72 43.18 0)
+    (property "Footprint" "Capacitor_SMD:C_0805_2012Metric_Pad1.18x1.45mm_HandSolder" (id 2) (at 45.72 43.18 0)
       (effects (font (size 1.27 1.27)) hide)
     )
@@
   (symbol (lib_id "Device:R_Small_US") (at 118.11 46.99 0) (unit 1)
     (in_bom yes) (on_board yes) (fields_autoplaced)
-    (property "Reference" "R?" (id 0) (at 119.761 46.1553 0)
+    (property "Reference" "R12" (id 0) (at 119.761 46.1553 0)
       (effects (font (size 1.27 1.27)) (justify left))
     )
@@
       (effects (font (size 1.27 1.27)) (justify left))
     )
-    (property "Footprint" "" (id 2) (at 118.11 46.99 0)
+    (property "Footprint" "Resistor_SMD:R_0805_2012Metric_Pad1.20x1.40mm_HandSolder" (id 2) (at 118.11 46.99 0)
       (effects (font (size 1.27 1.27)) hide)
     )
@@
   (symbol (lib_id "Regulator_Switching:TPS561201DDCR") (at 81.28 53.34 0) (unit 1)
     (in_bom yes) (on_board yes) (fields_autoplaced)
-    (property "Reference" "U?" (id 0) (at 81.28 24.291 0))
+    (property "Reference" "U5" (id 0) (at 81.28 24.291 0))
     (property "Value" "TPS561201DDCR" (id 1) (at 81.28 26.8279 0))
-    (property "Footprint" "" (id 2) (at 81.28 53.34 0)
+    (property "Footprint" "Package_TO_SOT_SMD:SOT-23-6" (id 2) (at 81.28 53.34 0)
       (effects (font (size 1.27 1.27)) hide)
     )
@@
   (symbol (lib_id "Device:C_Polarized_Small") (at 133.35 44.45 0) (unit 1)
     (in_bom yes) (on_board yes) (fields_autoplaced)
-    (property "Reference" "C?" (id 0) (at 135.509 43.0692 0)
+    (property "Reference" "C14" (id 0) (at 135.509 43.0692 0)
       (effects (font (size 1.27 1.27)) (justify left))
     )
@@
       (effects (font (size 1.27 1.27)) (justify left))
     )
-    (property "Footprint" "" (id 2) (at 133.35 44.45 0)
+    (property "Footprint" "Capacitor_SMD:C_0805_2012Metric_Pad1.18x1.45mm_HandSolder" (id 2) (at 133.35 44.45 0)
       (effects (font (size 1.27 1.27)) hide)
     )
@@
   (symbol (lib_id "Device:C_Small") (at 97.79 31.75 270) (unit 1)
     (in_bom yes) (on_board yes) (fields_autoplaced)
-    (property "Reference" "C?" (id 0) (at 97.7836 26.4881 90))
+    (property "Reference" "C13" (id 0) (at 97.7836 26.4881 90))
     (property "Value" "100nF" (id 1) (at 97.7836 29.025 90))
-    (property "Footprint" "" (id 2) (at 97.79 31.75 0)
+    (property "Footprint" "Capacitor_SMD:C_0805_2012Metric_Pad1.18x1.45mm_HandSolder" (id 2) (at 97.79 31.75 0)
       (effects (font (size 1.27 1.27)) hide)
     )
@@
   (symbol (lib_id "power:GND") (at 133.35 54.61 0) (unit 1)
     (in_bom yes) (on_board yes) (fields_autoplaced)
-    (property "Reference" "#PWR?" (id 0) (at 133.35 60.96 0)
+    (property "Reference" "#PWR037" (id 0) (at 133.35 60.96 0)
       (effects (font (size 1.27 1.27)) hide)
     )
